File: PCB.sch (EAGLE design)
At the start: 0 parts

Commit message: placed components
Parts:
- added GND-BAT, VBAT: (no value), SparkFun-Connectors:CONN_01OFFSET
- added GPS: (no value), con-lstb:MA04-1
- added GPS-DRIVER, GSM-DRIVER: (no value), semicon-smd-ipc:NPN-TRANSISTOR_SOT23
- added GPS-POWER, GSM-POWER: MOSFET-PCHANNEL, User-Submitted:MOSFET-PCHANNEL
- added R1, R2: 1k, eagle-ltspice:RR0402
- added R3, R4: 10k, eagle-ltspice:RR0603
- added RD1: 82k, eagle-ltspice:RR0402
- added RD2: 120k, eagle-ltspice:RR0402
- added S1: (no value), SparkFun-Retired:SWITCH-SPDTSMD
- added S2, S3: MOMENTARY-SWITCH-SPST-PTH-6.0MM, SparkFun-Switches:MOMENTARY-SWITCH-SPST-PTH-6.0MM
- added TBASE_L, TBASE_R: (no value), con-lstb:MA08-1
- added U$1: SIM800LMODULE, SIM800LMODULE:SIM800LMODULE
Connections:
- new net 0/FLASH: TBASE_R.4
- new net 16: TBASE_L.3
- new net 2/TXD1: TBASE_R.3
- new net 3.3V: TBASE_L.8
- new net 4/SDA: TBASE_R.5
- new net 5/SCL: TBASE_R.6
- new net 5V: GPS.4, TBASE_R.1
- new net A0: TBASE_L.2
- new net CS/TXD2: TBASE_L.7
- new net GND: GPS.1, TBASE_R.2
- new net MISO: TBASE_L.5
- new net MOSI/RXD2: TBASE_L.6
- new net RST: TBASE_L.1
- new net RX: GPS.3
- new net RXD: TBASE_R.7
- new net SCLK: TBASE_L.4
- new net TX: GPS.2
- new net TXD: TBASE_R.8
