File: PCB.sch (EAGLE design)
At the start: 19 parts

Commit message: finished scheme
Parts:
- removed S2, S3: MOMENTARY-SWITCH-SPST-PTH-6.0MM, SparkFun-Switches:MOMENTARY-SWITCH-SPST-PTH-6.0MM
- added BTN-GND, BTN1, BTN2, BTN3: (no value), SparkFun-Connectors:CONN_01OFFSET
Connections:
- removed net 16: TBASE_L.3
- removed net RX: GPS.3
- removed net TX: GPS.2
- new net N$1: S1.P, VBAT.1
- new net N$2: GPS-DRIVER.E, GPS-POWER.G, R4.1
- new net N$3: GSM-POWER.S, R3.1, RD1.2, S1.S
- new net N$4: GSM-POWER.D, U$1.VCC
- new net N$5: GSM-DRIVER.E, GSM-POWER.G, R3.2
- net 0/FLASH: now also BTN2.1
- net 2/TXD1: now also BTN3.1
- net 4/SDA: now also BTN1.1
- net 5/SCL: now also GPS-DRIVER.B, R1.1
- net 5V: now also GPS-POWER.D, GPS-POWER.S, R4.2
- net A0: now also RD1.1, RD2.2
- net CS/TXD2: now also GSM-DRIVER.B, R2.1
- net GND: now also BTN-GND.1, GND-BAT.1, GPS-DRIVER.C, GSM-DRIVER.C, R1.2, R2.2, RD2.1, U$1.GND
- net MISO: now also U$1.RX
- net MOSI/RXD2: now also U$1.TX
- net RST: now also TBASE_L.3
- net RXD: now also GPS.2
- net SCLK: now also U$1.RST
- net TXD: now also GPS.3
Other:
- moved on the sheet: GND-BAT, GPS, GPS-DRIVER, GPS-POWER, GSM-DRIVER, GSM-POWER, R1, R2, R3, R4, RD1, RD2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

Commit message: finished scheme
Parts:
- removed BTN-GND, BTN1, BTN2, BTN3: (no value), SparkFun-Connectors:CONN_01OFFSET
- added D2: (no value), SparkFun-LED:LED-RGB-CCPIRANHA
- added R10, R11, R9: 100, eagle-ltspice:RR0603
- added R5: 1k, eagle-ltspice:RR0603
- added R6: 330, eagle-ltspice:RR0603
- added R7: 220, eagle-ltspice:RR0603
- added R8: 470, eagle-ltspice:RR0603
- added S2, S3, S4, S5: MOMENTARY-SWITCH-SPST-SMD-6.0X3.5MM, SparkFun-Switches:MOMENTARY-SWITCH-SPST-SMD-6.0X3.5MM
Connections:
- new net GPS-VCC: GPS-POWER.D, GPS.4
- new net N$10: D2.RED, R10.1
- new net N$11: D2.GRN, R11.1
- new net N$6: R8.1, S4.2
- new net N$7: R6.1, S5.2
- new net N$8: R7.1, S2.2
- new net N$9: R9.1, S3.2
- net 0/FLASH: no longer BTN2.1
- net 2/TXD1: now also R11.2; no longer BTN3.1
- net 3.3V: now also R6.2, R7.2, R8.2, R9.2
- net 4/SDA: now also R10.2; no longer BTN1.1
- net 5V: no longer GPS-POWER.D, GPS.4
- net A0: now also R5.2, S2.1, S3.1, S4.1, S5.1
- net GND: now also D2.C, R5.1; no longer BTN-GND.1
