File: prototype#2_ESP32/PCB/PCB1.brd (EAGLE design)
At the start: 62.2 x 54.4 mm, 16 parts

Commit message: finished pcb for prototype 2
Parts:
- removed G1: SL-160AA/PR, battery:SL-160AA/PR
- removed IC1: (no value), SSFD - ESP32 WEMOS LOLIN CHINA W_BATT:SSFD_LOLIN32_WEMOS_CHINA_W_BATT
- added +BAT, -BAT: PTR1PAD1-13Y, testpad:P1-13Y
- added U$2: TTGO-T-DISPLAYFRAME, TTGO-TDisplay:TTGO-T-DISPLAY-OL
- moved R9 35.2 mm to (26.9, 70.9)
- moved S2 17.1 mm to (58.9, 69.2), turned to 270 degrees
- moved RD2 11.0 mm to (37.0, 95.1), turned to 180 degrees
- moved RD1 4.35 mm to (33.7, 95.1), turned to 180 degrees
- moved SV1 1.80 mm to (59.9, 57.4)
Connections:
- removed net CS/TXD2: GSM-DRIVER.1, IC1.23, R2.1
- removed net GPS_RXD: IC1.17, SV1.1
- removed net GPS_TXD: IC1.16, SV1.2
- new net 17/TX2: U$1.RX, U$2.13-G13-A14
- new net 18/TX1: SV1.2, U$2.33-G33-A5
- new net 4/GSM_EN: GSM-DRIVER.1, R2.1, U$2.25-G25-A18-DAC1
- net 5/SCL: now also U$2.26-G26-A19-DAC2; no longer IC1.4
- net 5V: now also U$2.5V; no longer IC1.5V
- net A0: now also U$2.2-G2-A12; no longer IC1.26
- net GND: now also -BAT.TP, U$2.GND_0, U$2.GND_1, U$2.GND_2, U$2.GND_3, U$2.GND_4; no longer G1.-
- net N$3: now also +BAT.TP; no longer G1.+
- net N$6: now also SV1.1, U$2.32-G32-A4; no longer IC1.18, U$1.RX
- net N$7: now also U$2.15-G15-A13; no longer IC1.19
- net N$8: now also S2.1, U$2.3V3_0, U$2.3V3_1; no longer IC1.3V3A, R9.2
- net N$9: now also R9.2, U$2.27-G27-A17; no longer IC1.25, S2.1
Routing:
- net GND: track 7.08 -> 89.2 mm, vias 0 -> 6
- net 5V: track 103.9 -> 39.3 mm
- net 17/TX2: track 0.00 -> 57.6 mm
- net GPS_TXD: track 51.4 -> 0.00 mm
- net GPS_RXD: track 45.8 -> 0.00 mm
- net CS/TXD2: track 39.8 -> 0.00 mm, vias 3 -> 0
- net 18/TX1: track 0.00 -> 39.3 mm
- net 4/GSM_EN: track 0.00 -> 38.0 mm, vias 0 -> 2
- net N$1: track 4.23 -> 35.5 mm, vias 0 -> 2
- net N$9: track 32.0 -> 8.06 mm, vias 0 -> 2
- net N$7: track 38.7 -> 57.6 mm
- net N$8: track 5.11 -> 14.1 mm
- net 5/SCL: track 21.2 -> 28.3 mm, vias 0 -> 2
- net VCC: track 35.5 -> 37.4 mm
- net N$6: track 36.4 -> 35.2 mm
Other:
- board size 62.2 x 54.4 mm -> 62.7 x 54.4 mm
