File: prototype#2_ESP32/PCB/PCB1.sch (EAGLE design)
At the start: 16 parts

Commit message: finished pcb for prototype 2
Parts:
- removed G1: SL-160AA/PR, battery:SL-160AA/PR
- removed IC1: (no value), SSFD - ESP32 WEMOS LOLIN CHINA W_BATT:SSFD_LOLIN32_WEMOS_CHINA_W_BATT
- added +BAT, -BAT: PTR1PAD1-13Y, testpad:PTR1PAD1-13Y
- added U$2: TTGO-T-DISPLAYFRAME, TTGO-TDisplay:TTGO-T-DISPLAYFRAME
Connections:
- removed net CS/TXD2: GSM-DRIVER.B, IC1.23, R2.1
- removed net GPS_RXD: IC1.17, SV1.1
- removed net GPS_TXD: IC1.16, SV1.2
- new net 17/TX2: U$1.RX, U$2.13/A14
- new net 18/TX1: SV1.2, U$2.33/A5
- new net 4/GSM_EN: GSM-DRIVER.B, R2.1, U$2.25/A18/DAC1
- net 5/SCL: now also U$2.26/A19/DAC2; no longer IC1.4
- net 5V: now also U$2.5V; no longer IC1.5V
- net A0: now also U$2.2/A12; no longer IC1.26
- net GND: now also -BAT.TP, U$2.GND; no longer G1.-
- net N$3: now also +BAT.TP; no longer G1.+
- net N$6: now also SV1.1, U$2.32/A4; no longer IC1.18, U$1.RX
- net N$7: now also U$2.15/A13; no longer IC1.19
- net N$8: now also S2.1, U$2.3V3; no longer IC1.3V3A, R9.2
- net N$9: now also R9.2, U$2.27/A17; no longer IC1.25, S2.1
Other:
- moved on the sheet: R9, S2
